Commit message: Created core URDF

File: description/robot_core.xacro (robot description, xacro)
@@ -21,35 +21,35 @@
         <parent link="base_link"/>
         <child link="chassis"/>
-        <origin xyz="-0.1 0 0"/>
+        <origin xyz="0 0 0"/>
     </joint>
     <link name="chassis">
         <visual>
-            <origin xyz="0.15 0 0.075"/>
+            <origin xyz="0.0 0.0 0.01"/>
             <geometry>
-                <box size="0.3 0.3 0.15"/>
+                <box size="0.180 0.180 0.06"/>
             </geometry>
             <material name="white"/>
         </visual>
         <collision>
-            <origin xyz="0.15 0 0.075"/>
+            <origin xyz="0.0 0 0.01"/>
             <geometry>
-                <box size="0.3 0.3 0.15"/>
+                <box size="0.18 0.18 0.06"/>
             </geometry>
         </collision>
-        <xacro:inertial_box mass="0.5" x="0.3" y="0.3" z="0.15">
-            <origin xyz="0.15 0 0.075" rpy="0 0 0"/>
+        <xacro:inertial_box mass="0.5" x="0.18" y="0.18" z="0.06">
+            <origin xyz="0.0 0 0.01" rpy="0 0 0"/>
         </xacro:inertial_box>
     </link>
-    <!-- LEFT WHEEL LINK -->
-    <joint name="left_wheel_joint" type="continuous">
+    <!-- LEFT WHEEL 1 LINK -->
+    <joint name="left_wheel_1_joint" type="continuous">
         <parent link="base_link"/>
-        <child link="left_wheel"/>
-        <origin xyz="0 0.175 0" rpy="-${pi/2} 0 0" />
+        <child link="left_wheel_1"/>
+        <origin xyz="0.05 0.120 0" rpy="-${pi/2} 0 0" />
         <axis xyz="0 0 1"/>
     </joint>
-    <link name="left_wheel">
+    <link name="left_wheel_1">
         <visual>
             <geometry>
-                <cylinder radius="0.05" length="0.04"/>
+                <cylinder radius="0.04" length="0.05"/>
             </geometry>
             <material name="blue"/>
@@ -57,22 +57,45 @@
         <collision>
             <geometry>
-                <cylinder radius="0.05" length="0.04"/>
+                <cylinder radius="0.04" length="0.05"/>
             </geometry>
         </collision>
-        <xacro:inertial_cylinder mass="0.1" length="0.04" radius="0.05">
+        <xacro:inertial_cylinder mass="0.1" length="0.05" radius="0.04">
             <origin xyz="0 0 0" rpy="0 0 0"/>
         </xacro:inertial_cylinder>
     </link>
-    <!-- RIGHT WHEEL LINK -->
-    <joint name="right_wheel_joint" type="continuous">
+        <!-- LEFT WHEEL 2 LINK -->
+        <joint name="left_wheel_2_joint" type="continuous">
+            <parent link="base_link"/>
+            <child link="left_wheel_2"/>
+            <origin xyz="-0.05 0.120 0" rpy="-${pi/2} 0 0" />
+            <axis xyz="0 0 1"/>
+        </joint>
+        <link name="left_wheel_2">
+            <visual>
+                <geometry>
+                    <cylinder radius="0.04" length="0.05"/>
+                </geometry>
+                <material name="blue"/>
+            </visual>
+            <collision>
+                <geometry>
+                    <cylinder radius="0.04" length="0.05"/>
+                </geometry>
+            </collision>
+            <xacro:inertial_cylinder mass="0.1" length="0.05" radius="0.04">
+                <origin xyz="0 0 0" rpy="0 0 0"/>
+            </xacro:inertial_cylinder>
+        </link>
+    <!-- RIGHT WHEEL 1 LINK -->
+    <joint name="right_wheel_1_joint" type="continuous">
         <parent link="base_link"/>
-        <child link="right_wheel"/>
-        <origin xyz="0 -0.175 0" rpy="${pi/2} 0 0" />
+        <child link="right_wheel_1"/>
+        <origin xyz="0.05 -0.120 0" rpy="${pi/2} 0 0" />
         <axis xyz="0 0 -1"/>
     </joint>
-    <link name="right_wheel">
+    <link name="right_wheel_1">
         <visual>
             <geometry>
-                <cylinder radius="0.05" length="0.04"/>
+                <cylinder radius="0.04" length="0.05"/>
             </geometry>
             <material name="blue"/>
@@ -80,32 +103,33 @@
         <collision>
             <geometry>
-                <cylinder radius="0.05" length="0.04"/>
+                <cylinder radius="0.04" length="0.05"/>
             </geometry>
         </collision>
-        <xacro:inertial_cylinder mass="0.1" length="0.04" radius="0.05">
+        <xacro:inertial_cylinder mass="0.1" length="0.05" radius="0.04">
             <origin xyz="0 0 0" rpy="0 0 0"/>
         </xacro:inertial_cylinder>
     </link>
-    <!-- CASTER WHEEL LINK -->
-    <joint name="caster_wheel_joint" type="fixed">
-        <parent link="chassis"/>
-        <child link="caster_wheel"/>
-        <origin xyz="0.24 0 0"/>
+    <!-- RIGHT WHEEL 2 LINK -->
+    <joint name="right_wheel_2_joint" type="continuous">
+        <parent link="base_link"/>
+        <child link="right_wheel_2"/>
+        <origin xyz="-.050 -0.120 0" rpy="${pi/2} 0 0" />
+        <axis xyz="0 0 -1"/>
     </joint>
-    <link name="caster_wheel">
+    <link name="right_wheel_2">
         <visual>
             <geometry>
-                <sphere radius="0.05"/>
+                <cylinder radius="0.04" length="0.05"/>
             </geometry>
-            <material name="black"/>
+            <material name="blue"/>
         </visual>
         <collision>
             <geometry>
-                <sphere radius="0.05"/>
+                <cylinder radius="0.04" length="0.05"/>
             </geometry>
         </collision>
-        <xacro:inertial_sphere mass="0.1" radius="0.05">
+        <xacro:inertial_cylinder mass="0.1" length="0.05" radius="0.04">
             <origin xyz="0 0 0" rpy="0 0 0"/>
-        </xacro:inertial_sphere>
+        </xacro:inertial_cylinder>
     </link>
 </robot>
