Commit message: working urdf in gazebo

File: description/robot.urdf.xacro (robot description, xacro)
@@ -2,3 +2,4 @@
 <robot xmlns:xacro="http://www.ros.org/wiki/xacro"  name="robot">
     <xacro:include filename="robot_core.xacro" />
+    <xacro:include filename="gazebo_control.xacro"/>
 </robot>

File: description/robot_core.xacro (robot description, xacro)
@@ -41,12 +41,15 @@
         </xacro:inertial_box>
     </link>
+    <gazebo reference="chassis">
+        <material>Gazebo/White</material>
+    </gazebo>
     <!-- LEFT WHEEL 1 LINK -->
-    <joint name="left_wheel_1_joint" type="continuous">
+    <joint name="left_wheel_joint" type="continuous">
         <parent link="base_link"/>
-        <child link="left_wheel_1"/>
+        <child link="left_wheel"/>
         <origin xyz="0.05 0.120 0" rpy="-${pi/2} 0 0" />
         <axis xyz="0 0 1"/>
     </joint>
-    <link name="left_wheel_1">
+    <link name="left_wheel">
         <visual>
             <geometry>
@@ -64,6 +67,9 @@
         </xacro:inertial_cylinder>
     </link>
+    <gazebo reference="left_wheel">
+        <material>Gazebo/Blue</material>
+    </gazebo>
         <!-- LEFT WHEEL 2 LINK -->
-        <joint name="left_wheel_2_joint" type="continuous">
+        <joint name="left_wheel_joint_2" type="continuous">
             <parent link="base_link"/>
             <child link="left_wheel_2"/>
@@ -87,12 +93,15 @@
             </xacro:inertial_cylinder>
         </link>
+        <gazebo reference="left_wheel_2">
+            <material>Gazebo/Blue</material>
+        </gazebo>
     <!-- RIGHT WHEEL 1 LINK -->
-    <joint name="right_wheel_1_joint" type="continuous">
+    <joint name="right_wheel_joint" type="continuous">
         <parent link="base_link"/>
-        <child link="right_wheel_1"/>
+        <child link="right_wheel"/>
         <origin xyz="0.05 -0.120 0" rpy="${pi/2} 0 0" />
         <axis xyz="0 0 -1"/>
     </joint>
-    <link name="right_wheel_1">
+    <link name="right_wheel">
         <visual>
             <geometry>
@@ -110,6 +119,9 @@
         </xacro:inertial_cylinder>
     </link>
+    <gazebo reference="right_wheel">
+        <material>Gazebo/Blue</material>
+    </gazebo>
     <!-- RIGHT WHEEL 2 LINK -->
-    <joint name="right_wheel_2_joint" type="continuous">
+    <joint name="right_wheel_joint_2" type="continuous">
         <parent link="base_link"/>
         <child link="right_wheel_2"/>
@@ -133,3 +145,6 @@
         </xacro:inertial_cylinder>
     </link>
+    <gazebo reference="right_wheel_2">
+        <material>Gazebo/Blue</material>
+    </gazebo>
 </robot>
